File: TPF/Master_0/case_master/case_master.kicad_sch (KiCad schematic)
At the start: 66 parts, among them J1 Jack, J2 Pul_0, J3 Pul_0, J4 Pul_0, J5 Vin_3v3, J7 NRF24L01, J8 USART, Q1 BC337, U1 LM7805_TO220, U2 AMS1117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

Commit message: Update gral
Other:
- note added: "Master"
- moved on the sheet: J2, J3, J4
Changed lines of the file:
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@@
 	(wire
 		(pts
-			(xy 227.33 152.4) (xy 227.33 156.21)
+			(xy 241.3 153.67) (xy 241.3 157.48)
 		)
 		(stroke
@@
 	(wire
 		(pts
-			(xy 255.27 152.4) (xy 255.27 156.21)
+			(xy 269.24 153.67) (xy 269.24 157.48)
 		)
 		(stroke
@@
 	(wire
 		(pts
-			(xy 240.03 152.4) (xy 240.03 156.21)
+			(xy 254 153.67) (xy 254 157.48)
 		)
 		(stroke
@@
 	(wire
 		(pts
-			(xy 224.79 152.4) (xy 224.79 156.21)
+			(xy 238.76 153.67) (xy 238.76 157.48)
 		)
 		(stroke
@@
 	(wire
 		(pts
-			(xy 257.81 152.4) (xy 257.81 156.21)
+			(xy 271.78 153.67) (xy 271.78 157.48)
 		)
 		(stroke
@@
 	(wire
 		(pts
-			(xy 242.57 152.4) (xy 242.57 156.21)
+			(xy 256.54 153.67) (xy 256.54 157.48)
 		)
 		(stroke
@@
 		)
 	)
+	(text "Master"
+		(exclude_from_sim no)
+		(at 192.278 189.738 0)
+		(effects
+			(font
+				(size 1.905 1.905)
+			)
+		)
+	)
 	(text "I_buzz = 30mA"
 		(exclude_from_sim no)
@@
 	(global_label "5v"
 		(shape input)
-		(at 255.27 156.21 270)
+		(at 269.24 157.48 270)
 		(fields_autoplaced yes)
 		(effects
@@
 		)
 		(property "Intersheetrefs" "${INTERSHEET_REFS}"
-			(at 255.27 161.3723 90)
+			(at 269.24 162.6423 90)
 			(effects
 				(font
@@
 	(global_label "5v"
 		(shape input)
-		(at 240.03 156.21 270)
+		(at 254 157.48 270)
 		(fields_autoplaced yes)
 		(effects
@@
 		)
 		(property "Intersheetrefs" "${INTERSHEET_REFS}"
-			(at 240.03 161.3723 90)
+			(at 254 162.6423 90)
 			(effects
 				(font
@@
 	(global_label "P0"
 		(shape input)
-		(at 227.33 156.21 270)
+		(at 241.3 157.48 270)
 		(fields_autoplaced yes)
 		(effects
@@
 		)
 		(property "Intersheetrefs" "${INTERSHEET_REFS}"
-			(at 227.33 161.6747 90)
+			(at 241.3 162.9447 90)
 			(effects
 				(font
@@
 	(global_label "P1"
 		(shape input)
-		(at 242.57 156.21 270)
+		(at 256.54 157.48 270)
 		(fields_autoplaced yes)
 		(effects
@@
 		)
 		(property "Intersheetrefs" "${INTERSHEET_REFS}"
-			(at 242.57 161.6747 90)
+			(at 256.54 162.9447 90)
 			(effects
 				(font
@@
 	(global_label "5v"
 		(shape input)
-		(at 224.79 156.21 270)
+		(at 238.76 157.48 270)
 		(fields_autoplaced yes)
 		(effects
@@
 		)
 		(property "Intersheetrefs" "${INTERSHEET_REFS}"
-			(at 224.79 161.3723 90)
+			(at 238.76 162.6423 90)
 			(effects
 				(font
@@
 	(global_label "P2"
 		(shape input)
-		(at 257.81 156.21 270)
+		(at 271.78 157.48 270)
 		(fields_autoplaced yes)
 		(effects
@@
 		)
 		(property "Intersheetrefs" "${INTERSHEET_REFS}"
-			(at 257.81 161.6747 90)
+			(at 271.78 162.9447 90)
 			(effects
 				(font
@@
 	(symbol
 		(lib_id "Connector:Conn_01x02_Pin")
-		(at 257.81 147.32 270)
+		(at 271.78 148.59 270)
 		(unit 1)
 		(exclude_from_sim no)
@@
 		(fields_autoplaced yes)
 		(property "Reference" "J4"
-			(at 259.08 146.6849 90)
+			(at 273.05 147.9549 90)
 			(effects
 				(font
@@
 		)
 		(property "Value" "Pul_0"
-			(at 259.08 149.2249 90)
+			(at 273.05 150.4949 90)
 			(effects
 				(font
@@
 		)
 		(property "Footprint" "Connector_JST:JST_XA_B02B-XASK-1_1x02_P2.50mm_Vertical"
-			(at 257.81 147.32 0)
+			(at 271.78 148.59 0)
 			(effects
 				(font
@@
 		)
 		(property "Datasheet" "~"
-			(at 257.81 147.32 0)
+			(at 271.78 148.59 0)
 			(effects
 				(font
@@
 		)
 		(property "Description" "Generic connector, single row, 01x02, script generated"
-			(at 257.81 147.32 0)
+			(at 271.78 148.59 0)
 			(effects
 				(font
@@
 	(symbol
 		(lib_id "Connector:Conn_01x02_Pin")
-		(at 242.57 147.32 270)
+		(at 256.54 148.59 270)
 		(unit 1)
 		(exclude_from_sim no)
@@
 		(fields_autoplaced yes)
 		(property "Reference" "J3"
-			(at 243.84 146.6849 90)
+			(at 257.81 147.9549 90)
 			(effects
 				(font
@@
 		)
 		(property "Value" "Pul_0"
-			(at 243.84 149.2249 90)
+			(at 257.81 150.4949 90)
 			(effects
 				(font
@@
 		)
 		(property "Footprint" "Connector_JST:JST_XA_B02B-XASK-1_1x02_P2.50mm_Vertical"
-			(at 242.57 147.32 0)
+			(at 256.54 148.59 0)
 			(effects
 				(font
@@
 		)
 		(property "Datasheet" "~"
-			(at 242.57 147.32 0)
+			(at 256.54 148.59 0)
 			(effects
 				(font
@@
 		)
 		(property "Description" "Generic connector, single row, 01x02, script generated"
-			(at 242.57 147.32 0)
+			(at 256.54 148.59 0)
 			(effects
 				(font
@@
 	(symbol
 		(lib_id "Connector:Conn_01x02_Pin")
-		(at 227.33 147.32 270)
+		(at 241.3 148.59 270)
 		(unit 1)
 		(exclude_from_sim no)
@@
 		(fields_autoplaced yes)
 		(property "Reference" "J2"
-			(at 228.6 146.6849 90)
+			(at 242.57 147.9549 90)
 			(effects
 				(font
@@
 		)
 		(property "Value" "Pul_0"
-			(at 228.6 149.2249 90)
+			(at 242.57 150.4949 90)
 			(effects
 				(font
@@
 		)
 		(property "Footprint" "Connector_JST:JST_XA_B02B-XASK-1_1x02_P2.50mm_Vertical"
-			(at 227.33 147.32 0)
+			(at 241.3 148.59 0)
 			(effects
 				(font
@@
 		)
 		(property "Datasheet" "~"
-			(at 227.33 147.32 0)
+			(at 241.3 148.59 0)
 			(effects
 				(font
@@
 		)
 		(property "Description" "Generic connector, single row, 01x02, script generated"
-			(at 227.33 147.32 0)
+			(at 241.3 148.59 0)
 			(effects
 				(font
