File: TPF/SLAVE_0/Kicad_project/case/case.kicad_sch (KiCad schematic)
At the start: 60 parts, among them J1 Jack, J10 DHT22, J11 Sigs, J12 Vin_5v, J13 Analog_aux, J14 Vin_5v, J15 Sens_caud, J16 Vin_5v, J17 Aux, J18 Vin_5v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

Commit message: Update gral
Other:
- note added: "Slave"
Changed lines of the file:
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@@
+		)
+	)
+	(text "Slave"
+		(exclude_from_sim no)
+		(at 191.262 189.738 0)
+		(effects
+			(font
+				(size 1.905 1.905)
+			)
 		)
 	)
